Commit message: feat: Migrate entire stack from Humble+Gazebo Classic to Jazzy+Gazebo Harmonic (2026)
BREAKING CHANGES - Full technology stack modernization:

Simulation:
- Gazebo Classic (EOL 2025) → Gazebo Harmonic (LTS, EOL 2029)
- SDF world format (.world → .sdf) with gz-sim system plugins
- Sensor plugins: libgazebo_ros_* → native gz-sim sensor definitions
- Spawn: gazebo_ros spawn_entity → ros_gz_sim create
- Topic bridge: embedded ROS plugins → ros_gz_bridge parameter_bridge

ROS 2:
- Distribution: Humble → Jazzy Jalisco (LTS, EOL 2029)
- Docker base: osrf/ros:humble-desktop-full → osrf/ros:jazzy-desktop-full

Navigation:
- Local controller: DWB (dwb_core::DWBLocalPlanner) → MPPI (nav2_mppi_controller::MPPIController)
- MPPI provides 45-50% perf improvement via Eigen, sampling-based trajectory optimization
- Critics: ConstraintCritic, CostCritic, GoalCritic, PathAlignCritic, PathFollowCritic, etc.

Sensors (Gazebo Harmonic native):
- LiDAR: libgazebo_ros_ray_sensor → gz-sim gpu_lidar sensor
- Camera: libgazebo_ros_camera → gz-sim camera sensor
- IMU: libgazebo_ros_imu_sensor → gz-sim imu sensor
- Diff Drive: libgazebo_ros_diff_drive → gz-sim-diff-drive-system
- Joint States: auto → gz-sim-joint-state-publisher-system

Localization:
- robot_localization updated for Jazzy Lifecycle Node support

Documentation updated with latest tech versions and interview prep.

File: ros2_ws/src/auto_robot_description/urdf/camera.xacro (robot description, xacro)
@@ -30,10 +30,12 @@
   </joint>
   <link name="camera_link_optical"/>
+  <!-- Gazebo Harmonic Camera Sensor -->
+  <!-- Topics are bridged to ROS 2 via ros_gz_bridge in the launch file -->
   <gazebo reference="camera_link">
-    <material>Gazebo/Red</material>
     <sensor name="camera" type="camera">
-      <pose> 0 0 0 0 0 0 </pose>
+      <pose>0 0 0 0 0 0</pose>
       <visualize>true</visualize>
       <update_rate>30</update_rate>
+      <topic>camera/image_raw</topic>
       <camera>
         <horizontal_fov>1.089</horizontal_fov>
@@ -53,13 +55,4 @@
         </noise>
       </camera>
-      <plugin name="camera_controller" filename="libgazebo_ros_camera.so">
-        <frame_name>camera_link_optical</frame_name>
-        <camera_name>camera</camera_name>
-        <ros>
-          <namespace>/</namespace>
-          <argument>~/image_raw:=camera/image_raw</argument>
-          <argument>~/camera_info:=camera/camera_info</argument>
-        </ros>
-      </plugin>
     </sensor>
   </gazebo>

File: ros2_ws/src/auto_robot_description/urdf/gazebo_control.xacro (robot description, xacro)
@@ -1,28 +1,32 @@
 <?xml version="1.0"?>
 <robot xmlns:xacro="http://www.ros.org/wiki/xacro">
+  <!-- Gazebo Harmonic Differential Drive Plugin (gz-sim-diff-drive-system) -->
+  <!-- Note: In Gazebo Harmonic, plugins are specified in the URDF/SDF model.
+       The ros_gz_bridge is used to bridge Gazebo transport topics to ROS 2.
+       publish_odom_tf is set to false because robot_localization EKF handles this. -->
   <gazebo>
-    <plugin name="diff_drive" filename="libgazebo_ros_diff_drive.so">
+    <plugin filename="gz-sim-diff-drive-system" name="gz::sim::systems::DiffDrive">
       <!-- Wheel Information -->
       <left_joint>left_wheel_joint</left_joint>
       <right_joint>right_wheel_joint</right_joint>
       <wheel_separation>0.35</wheel_separation>
-      <wheel_diameter>0.10</wheel_diameter>
+      <wheel_radius>0.05</wheel_radius>
       <!-- Limits -->
-      <max_wheel_torque>200</max_wheel_torque>
-      <max_wheel_acceleration>10.0</max_wheel_acceleration>
+      <max_linear_acceleration>2.5</max_linear_acceleration>
       <!-- Output -->
-      <odometry_frame>odom</odometry_frame>
-      <robot_base_frame>base_footprint</robot_base_frame>
+      <frame_id>odom</frame_id>
+      <child_frame_id>base_footprint</child_frame_id>
       <publish_odom>true</publish_odom>
       <publish_odom_tf>false</publish_odom_tf>
       <publish_wheel_tf>true</publish_wheel_tf>
-      <odometry_topic>odom_raw</odometry_topic>
-      <ros>
-        <namespace>/</namespace>
-        <remapping>cmd_vel:=cmd_vel</remapping>
-        <remapping>odom:=odom_raw</remapping>
-      </ros>
-      <!-- Update rate -->
-      <update_rate>50</update_rate>
+      <odom_topic>odom_raw</odom_topic>
+      <topic>cmd_vel</topic>
+      <odom_publish_frequency>50</odom_publish_frequency>
+    </plugin>
+  </gazebo>
+  <!-- Joint State Publisher Plugin for Gazebo Harmonic -->
+  <gazebo>
+    <plugin filename="gz-sim-joint-state-publisher-system" name="gz::sim::systems::JointStatePublisher">
+      <topic>joint_states</topic>
     </plugin>
   </gazebo>

File: ros2_ws/src/auto_robot_description/urdf/imu.xacro (robot description, xacro)
@@ -22,72 +22,24 @@
     </xacro:inertial_box>
   </link>
+  <!-- Gazebo Harmonic IMU Sensor -->
+  <!-- Topics are bridged to ROS 2 via ros_gz_bridge in the launch file -->
   <gazebo reference="imu_link">
-    <material>Gazebo/Cyan</material>
     <sensor name="imu_sensor" type="imu">
       <always_on>true</always_on>
       <update_rate>50</update_rate>
       <visualize>false</visualize>
+      <topic>imu/data</topic>
       <imu>
         <angular_velocity>
-          <x>
-            <noise type="gaussian">
-              <mean>0.0</mean>
-              <stddev>2e-4</stddev>
-              <bias_mean>0.0000075</bias_mean>
-              <bias_stddev>0.0000008</bias_stddev>
-            </noise>
-          </x>
-          <y>
-            <noise type="gaussian">
-              <mean>0.0</mean>
-              <stddev>2e-4</stddev>
-              <bias_mean>0.0000075</bias_mean>
-              <bias_stddev>0.0000008</bias_stddev>
-            </noise>
-          </y>
-          <z>
-            <noise type="gaussian">
-              <mean>0.0</mean>
-              <stddev>2e-4</stddev>
-              <bias_mean>0.0000075</bias_mean>
-              <bias_stddev>0.0000008</bias_stddev>
-            </noise>
-          </z>
+          <x><noise type="gaussian"><mean>0.0</mean><stddev>2e-4</stddev></noise></x>
+          <y><noise type="gaussian"><mean>0.0</mean><stddev>2e-4</stddev></noise></y>
+          <z><noise type="gaussian"><mean>0.0</mean><stddev>2e-4</stddev></noise></z>
         </angular_velocity>
         <linear_acceleration>
-          <x>
-            <noise type="gaussian">
-              <mean>0.0</mean>
-              <stddev>1.7e-2</stddev>
-              <bias_mean>0.1</bias_mean>
-              <bias_stddev>0.001</bias_stddev>
-            </noise>
-          </x>
-          <y>
-            <noise type="gaussian">
-              <mean>0.0</mean>
-              <stddev>1.7e-2</stddev>
-              <bias_mean>0.1</bias_mean>
-              <bias_stddev>0.001</bias_stddev>
-            </noise>
-          </y>
-          <z>
-            <noise type="gaussian">
-              <mean>0.0</mean>
-              <stddev>1.7e-2</stddev>
-              <bias_mean>0.1</bias_mean>
-              <bias_stddev>0.001</bias_stddev>
-            </noise>
-          </z>
+          <x><noise type="gaussian"><mean>0.0</mean><stddev>1.7e-2</stddev></noise></x>
+          <y><noise type="gaussian"><mean>0.0</mean><stddev>1.7e-2</stddev></noise></y>
+          <z><noise type="gaussian"><mean>0.0</mean><stddev>1.7e-2</stddev></noise></z>
         </linear_acceleration>
       </imu>
-      <plugin name="imu_plugin" filename="libgazebo_ros_imu_sensor.so">
-        <ros>
-          <namespace>/</namespace>
-          <remapping>~/out:=imu/data</remapping>
-        </ros>
-        <initial_orientation_as_reference>false</initial_orientation_as_reference>
-        <frame_name>imu_link</frame_name>
-      </plugin>
     </sensor>
   </gazebo>

File: ros2_ws/src/auto_robot_description/urdf/lidar.xacro (robot description, xacro)
@@ -22,11 +22,13 @@
     </xacro:inertial_cylinder>
   </link>
+  <!-- Gazebo Harmonic GPU LiDAR Sensor -->
+  <!-- Topics are bridged to ROS 2 via ros_gz_bridge in the launch file -->
   <gazebo reference="laser_frame">
-    <material>Gazebo/Red</material>
-    <sensor name="laser" type="ray">
-      <pose> 0 0 0 0 0 0 </pose>
+    <sensor name="gpu_lidar" type="gpu_lidar">
+      <pose>0 0 0 0 0 0</pose>
       <visualize>false</visualize>
       <update_rate>10</update_rate>
-      <ray>
+      <topic>scan</topic>
+      <lidar>
         <scan>
           <horizontal>
@@ -47,12 +49,5 @@
           <stddev>0.008</stddev>
         </noise>
-      </ray>
-      <plugin name="laser_controller" filename="libgazebo_ros_ray_sensor.so">
-        <ros>
-          <argument>~/out:=scan</argument>
-        </ros>
-        <output_type>sensor_msgs/LaserScan</output_type>
-        <frame_name>laser_frame</frame_name>
-      </plugin>
+      </lidar>
     </sensor>
   </gazebo>
